File: kicad-project-v1/usb_atmega32u2_rfm12b.kicad_pcb (KiCad board)
At the start: 2 copper layers, 57.8 x 34.3 mm, 19 parts, among them K1 CONN_3, P1 CONN_7, P2 CONN_1, P3 CONN_4, P4 CONN_6, SW1 HWB, SW2 RESET, U1 ATMEGA32U2, U2 RFM12, U3 USBCONN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

Commit message: Added pull-up resistors on HWB and RESET.
Parts:
- added R4: 3k, SM0805, F.Cu at (107.3, 73.9)
- added R5: 3k, SM0805, F.Cu at (87.2, 46.5)
Routing:
- net /RESET: track 23.0 -> 27.2 mm
- net /VCC: track 117.8 -> 120.9 mm
- net N-0000031: track 19.3 -> 21.7 mm
